Commit message: Updated

File: src/auv_core/urdf/orca4_description.urdf (robot description, URDF)
Before this commit: robot orca4, 8 links, 7 joints
Links:
- removed link downward_camera_link
- added link imu_link; collision box ; visual box 
- added link left_camera_link, mass 0.001; visual cylinder length=0.135 radius=0.0275
- added link right_camera_link, mass 0.001; visual cylinder length=0.135 radius=0.0275
- link base_link: mass 12.036 -> 10.036; geometry collision box size=0.457 0.338 0.06506286173008947; visual mesh filename=package://simulation/models/orca4_ign/meshes/bluerov2.dae scale=0.025 0.025 0.025
- link thruster1: geometry visual mesh filename=package://simulation/models/orca4_ign/meshes/t200-cw-prop.d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
- link thruster2: geometry visual mesh filename=package://simulation/models/orca4_ign/meshes/t200-ccw-prop.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
- link thruster3: geometry visual mesh filename=package://simulation/models/orca4_ign/meshes/t200-ccw-prop.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
- link thruster4: geometry visual mesh filename=package://simulation/models/orca4_ign/meshes/t200-cw-prop.d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
- link thruster5: geometry visual mesh filename=package://simulation/models/orca4_ign/meshes/t200-ccw-prop.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
- link thruster6: geometry visual mesh filename=package://simulation/models/orca4_ign/meshes/t200-cw-prop.d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
Joints:
- removed joint downward_camera_joint
- added joint imu_joint: type fixed, parent base_link, child imu_link, origin xyz=0 0 0.01
- added joint left_camera_joint: type fixed, parent base_link, child left_camera_link, origin xyz=0.15 0.2 -0.0675 rpy=0 0 1.5707963267948966
- added joint right_camera_joint: type fixed, parent base_link, child right_camera_link, origin xyz=0.15 -0.2 -0.0675 rpy=0 0 -1.5707963267948966
- joint thruster1_joint: axis 0 0 1 -> 0 0 -1; limit effort=100 velocity=300 -> lower=-1e+12 upper=1e+12 effort=-1 velocity=-1; origin xyz=0.14 -0.092 0 rpy=-1.5708 1.5708 -0.7854 -> xyz=0.14 -0.092 0 rpy=-1.5707963267948966 1.5707963267948966 -0.7853981633974483
- joint thruster2_joint: axis 0 0 1 -> 0 0 -1; limit effort=100 velocity=300 -> lower=-1e+12 upper=1e+12 effort=-1 velocity=-1; origin xyz=0.14 0.092 0 rpy=-1.5708 1.5708 -2.3562 -> xyz=0.14 0.092 0 rpy=-1.5707963267948966 1.5707963267948966 -2.356194490192345
- joint thruster3_joint: axis 0 0 1 -> 0 0 -1; limit effort=100 velocity=300 -> lower=-1e+12 upper=1e+12 effort=-1 velocity=-1; origin xyz=-0.14 -0.092 0 rpy=-1.5708 1.5708 0.7854 -> xyz=-0.14 -0.092 0 rpy=-1.5707963267948966 1.5707963267948966 0.7853981633974483
- joint thruster4_joint: axis 0 0 1 -> 0 0 -1; limit effort=100 velocity=300 -> lower=-1e+12 upper=1e+12 effort=-1 velocity=-1; origin xyz=-0.14 0.092 0 rpy=-1.5708 1.5708 2.3562 -> xyz=-0.14 0.092 0 rpy=-1.5707963267948966 1.5707963267948966 2.356194490192345
- joint thruster5_joint: axis 0 0 1 -> 0 0 -1; limit effort=100 velocity=300 -> lower=-1e+12 upper=1e+12 effort=-1 velocity=-1
- joint thruster6_joint: axis 0 0 1 -> 0 0 -1; limit effort=100 velocity=300 -> lower=-1e+12 upper=1e+12 effort=-1 velocity=-1

Commit message: Updated

File: src/auv_core/urdf/orca4_description.urdf (robot description, URDF)
Before this commit: robot orca4_ign, 10 links, 9 joints
Links:
- added link downward_camera_link, mass 0.001
- added link forward_camera_link, mass 0.001
- link imu_link: mass None -> 0.001; geometry collision box size=0.01 0.01 0.01; visual box size=0.01 0.01 0.01
Joints:
- added joint downward_camera_joint: type fixed, parent base_link, child downward_camera_link, origin xyz=0.15 0 -0.05 rpy=0 0.3 0
- added joint forward_camera_joint: type fixed, parent base_link, child forward_camera_link, origin xyz=0.15 0 0 rpy=0 0 0
- joint imu_joint: origin xyz=0 0 0.01 -> xyz=0 0 0.01 rpy=0 0 0

Commit message: Updated

File: src/auv_core/urdf/orca4_description.urdf (robot description, URDF)
Before this commit: robot orca4_ign, 12 links, 11 joints
Links:
- link base_link: geometry collision box size=0.457 0.338 0.06506286173008947; visual mesh filename=package://auv_core/meshes/bluerov2.dae scale=0.025 0.025 0.025
- link downward_camera_link: geometry visual cylinder length=0.05 radius=0.02
- link forward_camera_link: geometry visual cylinder length=0.05 radius=0.02
- link thruster1: geometry visual mesh filename=package://auv_core/meshes/t200-cw-prop.dae
- link thruster2: geometry visual mesh filename=package://auv_core/meshes/t200-ccw-prop.dae
- link thruster3: geometry visual mesh filename=package://auv_core/meshes/t200-ccw-prop.dae
- link thruster4: geometry visual mesh filename=package://auv_core/meshes/t200-cw-prop.dae
- link thruster5: geometry visual mesh filename=package://auv_core/meshes/t200-ccw-prop.dae
- link thruster6: geometry visual mesh filename=package://auv_core/meshes/t200-cw-prop.dae
Joints:
- joint downward_camera_joint: origin xyz=0.15 0 -0.05 rpy=0 0.3 0 -> xyz=0 0 -0.1 rpy=0 1.5707963267948966 0
- joint forward_camera_joint: origin xyz=0.15 0 0 rpy=0 0 0 -> xyz=0.2 0 0 rpy=0 0 0

Commit message: Updated

File: src/auv_core/urdf/orca4_description.urdf (robot description, URDF)
Before this commit: robot orca4_ign, 12 links, 11 joints
Links:
- removed link downward_camera_link
- removed link left_camera_link
- removed link right_camera_link
Joints:
- removed joint downward_camera_joint
- removed joint left_camera_joint
- removed joint right_camera_joint

Commit message: Updated

File: src/auv_core/urdf/orca4_description.urdf (robot description, URDF)
Before this commit: robot orca4_ign, 9 links, 8 joints
Links:
- link base_link: geometry collision box size=0.457 0.338 0.067; visual mesh filename=package://auv_core/meshes/bluerov2.dae scale=0.025 0.025 0.025

Commit message: Updated

File: src/auv_core/urdf/orca4_description.urdf (robot description, URDF)
Before this commit: robot orca4_ign, 9 links, 8 joints
Links:
- removed link forward_camera_link
- added link left_camera_link, mass 0.001; visual cylinder length=0.135 radius=0.0275
- added link right_camera_link, mass 0.001; visual cylinder length=0.135 radius=0.0275
- link base_link: geometry collision box size=0.457 0.338 0.06506286173008947; visual mesh filename=package://simulation/models/orca4_ign/meshes/bluerov2.dae scale=0.025 0.025 0.025
- link imu_link: mass 0.001 -> None; geometry collision box ; visual box 
- link thruster1: geometry visual mesh filename=package://simulation/models/orca4_ign/meshes/t200-cw-prop.d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
- link thruster2: geometry visual mesh filename=package://simulation/models/orca4_ign/meshes/t200-ccw-prop.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
- link thruster3: geometry visual mesh filename=package://simulation/models/orca4_ign/meshes/t200-ccw-prop.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
- link thruster4: geometry visual mesh filename=package://simulation/models/orca4_ign/meshes/t200-cw-prop.d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
- link thruster5: geometry visual mesh filename=package://simulation/models/orca4_ign/meshes/t200-ccw-prop.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
- link thruster6: geometry visual mesh filename=package://simulation/models/orca4_ign/meshes/t200-cw-prop.d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
Joints:
- removed joint forward_camera_joint
- added joint left_camera_joint: type fixed, parent base_link, child left_camera_link, origin xyz=0.15 0.2 -0.0675 rpy=0 0 1.5707963267948966
- added joint right_camera_joint: type fixed, parent base_link, child right_camera_link, origin xyz=0.15 -0.2 -0.0675 rpy=0 0 -1.5707963267948966
- joint imu_joint: origin xyz=0 0 0.01 rpy=0 0 0 -> xyz=0 0 0.01
